File: PCBs/AIAB hat.kicad_pcb (KiCad board)
At the start: 2 copper layers, 77.1 x 84.8 mm, 49 parts, among them IC1 4050D, M11 TerminalBlock_Altech_AK300-2_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, M12 TerminalBlock_Altech_AK300-2_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, U1 PCA9685, U2 AP2112K-3.3, U4 MPU-6050, X1 MICROSD

Commit message: Add files via upload
Parts:
- added GND: PinHeader_1x05_P2.54mm_Vertical, Connector_PinHeader_2.54mm:PinHeader_1x05_P2.54mm_Vertical, F.Cu at (182.4, 22.9)
- added JP3: , 3X04, F.Cu at (175.0, 21.3)
- added R11_5: 10K, RESPACK_4X0603, F.Cu at (160.8, 20.8)
- added SPI Cam: PinHeader_1x08_P2.54mm_Vertical, Connector_PinHeader_2.54mm:PinHeader_1x08_P2.54mm_Vertical, F.Cu at (162.1, 102.9)
- added VCC: PinHeader_1x05_P2.54mm_Vertical, Connector_PinHeader_2.54mm:PinHeader_1x05_P2.54mm_Vertical, F.Cu at (186.4, 22.9)
Routing:
- net (no net): track 3313.0 -> 3828.4 mm, vias 105 -> 136
Other:
- board size 77.1 x 84.8 mm -> 77.1 x 89.2 mm

Commit message: corrected pins
Routing:
- net (no net): track 3828.4 -> 3831.7 mm
Changed lines of the file:
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@@
   (via (at 144.145 73.025) (size 0.8) (drill 0.4) (layers "F.Cu" "B.Cu") (net 0))
   (segment (start 155.052 92.187) (end 154.94 92.075) (width 0.25) (layer "B.Cu") (net 0))
+  (segment (start 197.104 90.678) (end 198.12 89.662) (width 0.25) (layer "B.Cu") (net 0))
   (segment (start 198.12 74.676) (end 197.612 74.168) (width 0.25) (layer "B.Cu") (net 0))
   (segment (start 168.927 89.298) (end 168.927 92.885701) (width 0.25) (layer "B.Cu") (net 0))
@@
   (segment (start 152.654 92.71) (end 155.194 95.25) (width 0.25) (layer "B.Cu") (net 0))
   (segment (start 162.672 92.187) (end 162.56 92.075) (width 0.25) (layer "B.Cu") (net 0))
+  (segment (start 195.834 91.948) (end 197.104 90.678) (width 0.25) (layer "B.Cu") (net 0))
   (segment (start 170.18 57.785) (end 172.959 55.006) (width 0.25) (layer "B.Cu") (net 0))
   (segment (start 161.582396 80.301) (end 169.799 88.517604) (width 0.25) (layer "B.Cu") (net 0))
@@
   (segment (start 162.306 98.552) (end 164.338 96.52) (width 0.25) (layer "B.Cu") (net 0))
   (segment (start 169.164 19.558) (end 169.164 18.034) (width 0.25) (layer "B.Cu") (net 0))
-  (segment (start 195.834 91.948) (end 198.12 89.662) (width 0.25) (layer "B.Cu") (net 0))
   (segment (start 163.707299 89.666299) (end 164.211 90.17) (width 0.25) (layer "B.Cu") (net 0))
   (segment (start 141.605 78.105) (end 131.445 78.105) (width 0.25) (layer "B.Cu") (net 0))
@@
   (segment (start 166.37 46.355) (end 158.75 53.975) (width 0.25) (layer "B.Cu") (net 0))
   (segment (start 166.577 87.202001) (end 161.670999 82.296) (width 0.25) (layer "B.Cu") (net 0))
+  (segment (start 197.104 93.98) (end 197.104 90.678) (width 0.25) (layer "B.Cu") (net 0))
   (segment (start 159.004 104.648) (end 159.004 104.14) (width 0.25) (layer "B.Cu") (net 0))
   (segment (start 162.941 89.916) (end 161.163 88.138) (width 0.25) (layer "B.Cu") (net 0))
